File: tools/aepro/aepro_27C512.sch (EAGLE design)
At the start: 22 parts, among them IC1 MCP23017SP, IC2 MCP23008/P, U1 328P, Y1 16 MHz

Commit message: AEPRO rev 7
Connections:
- removed net N$12: CN1.RXD, U1.PD0(RXD)
- removed net N$3: R5.1, V1/2.Y
- new net N$11: CN1.RXD, U1.PD1(TXD)
- net GND: now also V1/2.A
- net N$4: now also R5.1, U1.PD3(INT1); no longer U1.PD4(XCK/T0), V1/2.A
- net N$6: now also U1.PD0(RXD); no longer U1.PD1(TXD)
Other:
- moved on the sheet: CN1, R1, R2, V1/2
Changed lines of the file:
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@@
 <drawing>
 <settings>
-<setting alwaysvectorfont="yes"/>
+<setting alwaysvectorfont="no"/>
 <setting verticaltext="up"/>
 </settings>
@@
 <attribute name="VALUE" x="51.816" y="-21.971" size="1.778" layer="96"/>
 </instance>
-<instance part="R1" gate="G$1" x="154.94" y="50.8" smashed="yes">
-<attribute name="NAME" x="154.94" y="52.324" size="1.778" layer="95" font="vector" align="bottom-center"/>
-<attribute name="VALUE" x="154.94" y="49.276" size="1.778" layer="96" font="vector" align="top-center"/>
-</instance>
-<instance part="R2" gate="G$1" x="154.94" y="40.64" smashed="yes">
-<attribute name="NAME" x="154.94" y="42.164" size="1.778" layer="95" font="vector" align="bottom-center"/>
-<attribute name="VALUE" x="154.94" y="39.116" size="1.778" layer="96" font="vector" align="top-center"/>
-</instance>
-<instance part="SUPPLY4" gate="G$1" x="170.18" y="53.34" smashed="yes">
-<attribute name="VALUE" x="170.18" y="56.134" size="1.778" layer="96" align="bottom-center"/>
+<instance part="R1" gate="G$1" x="172.72" y="55.88" smashed="yes">
+<attribute name="NAME" x="172.72" y="57.404" size="1.778" layer="95" font="vector" align="bottom-center"/>
+<attribute name="VALUE" x="172.72" y="54.356" size="1.778" layer="96" font="vector" align="top-center"/>
+</instance>
+<instance part="R2" gate="G$1" x="172.72" y="45.72" smashed="yes">
+<attribute name="NAME" x="172.72" y="47.244" size="1.778" layer="95" font="vector" align="bottom-center"/>
+<attribute name="VALUE" x="172.72" y="44.196" size="1.778" layer="96" font="vector" align="top-center"/>
+</instance>
+<instance part="SUPPLY4" gate="G$1" x="187.96" y="58.42" smashed="yes">
+<attribute name="VALUE" x="187.96" y="61.214" size="1.778" layer="96" align="bottom-center"/>
 </instance>
 <instance part="U1" gate="U1" x="-20.32" y="7.62" smashed="yes">
@@
 <attribute name="VALUE" x="-38.1" y="-30.48" size="1.778" layer="96"/>
 </instance>
-<instance part="CN1" gate="G$1" x="48.26" y="15.24" smashed="yes">
-<attribute name="NAME" x="40.64" y="23.876" size="1.27" layer="95"/>
-<attribute name="VALUE" x="40.64" y="2.54" size="1.27" layer="96"/>
+<instance part="CN1" gate="G$1" x="48.26" y="12.7" smashed="yes">
+<attribute name="NAME" x="40.64" y="21.336" size="1.27" layer="95"/>
+<attribute name="VALUE" x="40.64" y="0" size="1.27" layer="96"/>
 </instance>
 <instance part="D1" gate="D1" x="-68.58" y="25.4" smashed="yes">
@@
 <attribute name="VALUE" x="92.075" y="38.1" size="2.032" layer="96" rot="R90"/>
 </instance>
-<instance part="V1" gate="/2" x="106.68" y="43.18" smashed="yes" rot="R90">
-<attribute name="NAME" x="100.965" y="38.1" size="2.032" layer="95" rot="R90"/>
-<attribute name="VALUE" x="114.935" y="38.1" size="2.032" layer="96" rot="R90"/>
+<instance part="V1" gate="/2" x="144.78" y="40.64" smashed="yes">
+<attribute name="NAME" x="139.7" y="46.355" size="2.032" layer="95"/>
+<attribute name="VALUE" x="139.7" y="32.385" size="2.032" layer="96"/>
 </instance>
 <instance part="V1" gate="/3" x="144.78" y="22.86" smashed="yes">
@@
 <bus name="I2C:SCL,SDA">
 <segment>
-<wire x1="144.78" y1="50.8" x2="144.78" y2="40.64" width="0.762" layer="92"/>
-<label x="134.62" y="50.8" size="2.54" layer="95"/>
+<wire x1="162.56" y1="55.88" x2="162.56" y2="45.72" width="0.762" layer="92"/>
+<label x="152.4" y="55.88" size="2.54" layer="95"/>
 </segment>
 <segment>
@@
 <segment>
 <pinref part="R1" gate="G$1" pin="2"/>
-<wire x1="160.02" y1="50.8" x2="170.18" y2="50.8" width="0.1524" layer="91"/>
+<wire x1="177.8" y1="55.88" x2="187.96" y2="55.88" width="0.1524" layer="91"/>
 <pinref part="SUPPLY4" gate="G$1" pin="VCC"/>
-<wire x1="170.18" y1="50.8" x2="170.18" y2="53.34" width="0.1524" layer="91"/>
+<wire x1="187.96" y1="55.88" x2="187.96" y2="58.42" width="0.1524" layer="91"/>
 <pinref part="R2" gate="G$1" pin="2"/>
-<wire x1="160.02" y1="40.64" x2="170.18" y2="40.64" width="0.1524" layer="91"/>
-<wire x1="170.18" y1="40.64" x2="170.18" y2="50.8" width="0.1524" layer="91"/>
-<junction x="170.18" y="50.8"/>
+<wire x1="177.8" y1="45.72" x2="187.96" y2="45.72" width="0.1524" layer="91"/>
+<wire x1="187.96" y1="45.72" x2="187.96" y2="55.88" width="0.1524" layer="91"/>
+<junction x="187.96" y="55.88"/>
 </segment>
 <segment>
@@
 <segment>
 <pinref part="CN1" gate="G$1" pin="VCC"/>
-<wire x1="38.1" y1="15.24" x2="22.86" y2="15.24" width="0.1524" layer="91"/>
+<wire x1="38.1" y1="12.7" x2="22.86" y2="12.7" width="0.1524" layer="91"/>
 <pinref part="SUPPLY6" gate="G$1" pin="VCC"/>
-<wire x1="22.86" y1="15.24" x2="22.86" y2="22.86" width="0.1524" layer="91"/>
+<wire x1="22.86" y1="12.7" x2="22.86" y2="22.86" width="0.1524" layer="91"/>
 </segment>
 <segment>
@@
 <segment>
 <pinref part="R2" gate="G$1" pin="1"/>
-<wire x1="144.78" y1="40.64" x2="149.86" y2="40.64" width="0.1524" layer="91"/>
+<wire x1="162.56" y1="45.72" x2="167.64" y2="45.72" width="0.1524" layer="91"/>
 </segment>
 <segment>
@@
 <segment>
 <pinref part="R1" gate="G$1" pin="1"/>
-<wire x1="149.86" y1="50.8" x2="144.78" y2="50.8" width="0.1524" layer="91"/>
+<wire x1="167.64" y1="55.88" x2="162.56" y2="55.88" width="0.1524" layer="91"/>
 </segment>
 <segment>
@@
 <segment>
 <pinref part="GND6" gate="1" pin="GND"/>
-<wire x1="25.4" y1="-5.08" x2="25.4" y2="20.32" width="0.1524" layer="91"/>
+<wire x1="25.4" y1="-5.08" x2="25.4" y2="17.78" width="0.1524" layer="91"/>
 <pinref part="CN1" gate="G$1" pin="GND"/>
-<wire x1="25.4" y1="20.32" x2="38.1" y2="20.32" width="0.1524" layer="91"/>
+<wire x1="25.4" y1="17.78" x2="38.1" y2="17.78" width="0.1524" layer="91"/>
 </segment>
 <segment>
@@
 <wire x1="157.48" y1="-7.62" x2="157.48" y2="-5.08" width="0.1524" layer="91"/>
 <junction x="157.48" y="-5.08"/>
+<pinref part="V1" gate="/2" pin="A"/>
+<wire x1="134.62" y1="40.64" x2="129.54" y2="40.64" width="0.1524" layer="91"/>
+<wire x1="129.54" y1="40.64" x2="129.54" y2="22.86" width="0.1524" layer="91"/>
+<junction x="129.54" y="22.86"/>
 </segment>
 <segment>
@@
 <segment>
 <wire x1="15.24" y1="30.48" x2="68.58" y2="30.48" width="0.1524" layer="91"/>
-<wire x1="15.24" y1="30.48" x2="15.24" y2="0" width="0.1524" layer="91"/>
-<pinref part="U1" gate="U1" pin="PD4(XCK/T0)"/>
-<wire x1="15.24" y1="0" x2="2.54" y2="0" width="0.1524" layer="91"/>
+<wire x1="15.24" y1="30.48" x2="15.24" y2="2.54" width="0.1524" layer="91"/>
 <pinref part="U$1" gate="G$1" pin="!CE"/>
 <wire x1="73.66" y1="15.24" x2="68.58" y2="15.24" width="0.1524" layer="91"/>
@@
 <wire x1="68.58" y1="30.48" x2="106.68" y2="30.48" width="0.1524" layer="91"/>
 <junction x="68.58" y="30.48"/>
-<pinref part="V1" gate="/2" pin="A"/>
-<wire x1="106.68" y1="30.48" x2="106.68" y2="33.02" width="0.1524" layer="91"/>
+<pinref part="R5" gate="G$1" pin="1"/>
+<wire x1="106.68" y1="30.48" x2="106.68" y2="53.34" width="0.1524" layer="91"/>
+<pinref part="U1" gate="U1" pin="PD3(INT1)"/>
+<wire x1="2.54" y1="2.54" x2="15.24" y2="2.54" width="0.1524" layer="91"/>
 </segment>
 </net>
@@
 <net name="N$6" class="0">
 <segment>
-<pinref part="U1" gate="U1" pin="PD1(TXD)"/>
-<wire x1="17.78" y1="7.62" x2="2.54" y2="7.62" width="0.1524" layer="91"/>
-<wire x1="17.78" y1="7.62" x2="17.78" y2="12.7" width="0.1524" layer="91"/>
+<pinref part="U1" gate="U1" pin="PD0(RXD)"/>
 <pinref part="CN1" gate="G$1" pin="TXD"/>
-<wire x1="17.78" y1="12.7" x2="38.1" y2="12.7" width="0.1524" layer="91"/>
+<wire x1="38.1" y1="10.16" x2="2.54" y2="10.16" width="0.1524" layer="91"/>
 </segment>
 </net>
@@
 <junction x="-50.8" y="99.06"/>
 <pinref part="CN1" gate="G$1" pin="RTS"/>
-<wire x1="38.1" y1="7.62" x2="35.56" y2="7.62" width="0.1524" layer="91"/>
-<wire x1="35.56" y1="7.62" x2="35.56" y2="40.64" width="0.1524" layer="91"/>
+<wire x1="38.1" y1="5.08" x2="35.56" y2="5.08" width="0.1524" layer="91"/>
+<wire x1="35.56" y1="5.08" x2="35.56" y2="40.64" width="0.1524" layer="91"/>
 <wire x1="35.56" y1="40.64" x2="-45.72" y2="40.64" width="0.1524" layer="91"/>
 <junction x="-45.72" y="40.64"/>
@@
 </segment>
 </net>
-<net name="N$12" class="0">
-<segment>
-<pinref part="CN1" gate="G$1" pin="RXD"/>
-<pinref part="U1" gate="U1" pin="PD0(RXD)"/>
-<wire x1="38.1" y1="10.16" x2="2.54" y2="10.16" width="0.1524" layer="91"/>
-</segment>
-</net>
 <net name="N$13" class="0">
 <segment>
@@
 </segment>
 </net>
-<net name="N$3" class="0">
-<segment>
-<pinref part="V1" gate="/2" pin="Y"/>
-<pinref part="R5" gate="G$1" pin="1"/>
-</segment>
-</net>
 <net name="N$8" class="0">
 <segment>
@@
 </segment>
 </net>
+<net name="N$11" class="0">
+<segment>
+<pinref part="U1" gate="U1" pin="PD1(TXD)"/>
+<pinref part="CN1" gate="G$1" pin="RXD"/>
+<wire x1="2.54" y1="7.62" x2="38.1" y2="7.62" width="0.1524" layer="91"/>
+</segment>
+</net>
