File: tools/sercon/sercon.sch (EAGLE design)
At the start: 13 parts, among them IC1 ATMEGA644-10PU

Commit message: AEPRO rev 7
Parts:
- removed U1, U2: (no value), SparkFun-IC-Logic:74595
- added U$4, U$5: 74595, wntrmute:74595
- C1: value (none) -> 0.1µF
- CN1: value (none) -> FTDI
- Y1: value (none) -> 16MHz
Connections:
- new net N$48: IC1.PCINT4/ADC4_PA4, U$5.RCK
- new net N$49: IC1.PCINT6/ADC6_PA6, U$5.G
- new net N$50: IC1.PCINT5/ADC5_PA5, U$4.G
- net GND: now also U$3.GND, U$4.GND, U$5.GND; no longer U$3.VCC, U1.GND, U2.GND
- net N$10: now also U$4.QE; no longer U1.QE
- net N$11: now also U$4.QF; no longer U1.QF
- net N$12: now also U$4.QG; no longer U1.QG
- net N$13: now also U$4.QH; no longer U1.QH
- net N$29: now also U$5.QA; no longer U2.QA
- net N$3: now also U$4.SCL, U$5.SCL
- net N$40: now also IC1.PCINT0/ADC0_PA0, U$4.SER; no longer IC1.PCINT22/TOSC1_PC6, U1.SER
- net N$41: now also IC1.PCINT1/ADC1_PA1, U$5.SER; no longer IC1.PCINT23/TOSC2_PC7, U2.SER
- net N$42: now also IC1.PCINT2/ADC2_PA2, U$4.SCK, U$5.SCK; no longer IC1.PCINT27/INT1_PD3, U1.SCK, U2.SCK
- net N$43: now also IC1.PCINT3/ADC3_PA3, U$4.RCK; no longer IC1.PCINT26/INT0_PD2, U1.SCL, U2.SCL
- net N$44: now also U$5.QB; no longer U2.QB
- net N$45: now also U$5.QC; no longer U2.QC
- net N$46: now also U$5.QD; no longer U2.QD
- net N$6: now also U$4.QA; no longer U1.QA
- net N$7: now also U$4.QB; no longer U1.QB
- net N$8: now also U$4.QC; no longer U1.QC
- net N$9: now also U$4.QD; no longer U1.QD
- net VCC: now also U$3.VCC, U$4.VCC, U$5.VCC; no longer U$3.GND, U1.VCC
